File: hardware/pcb/eink_schematic.brd (EAGLE design)
At the start: 97.9 x 74.6 mm, 18 parts, among them J2 5.5x2.1mm Barrel, Q1 FDN340P, U1 NUCLEUM, U2 LTC3531ES6-3PBF, U4 MAX6326UR29+

Commit message: redid battery
Parts:
- added LOGO1: UMICH_SOLID_LARGE, logos:UMICH_SOLID_350MIL
- moved BATTERY 27.4 mm to (81.5, 34.0)
Connections:
- net ENABLE renamed !ENABLE
- net TC_BUSY renamed !TC_BUSY
- removed net N$6: J2.GND, J2.P$4
- net GND: now also J2.GND, J2.P$4
Routing:
- net N$6: track 6.10 -> 0.00 mm
- net GND: track 138.6 -> 143.9 mm
Other:
- outline, holes or cut-outs redrawn
- board text added: "5V"
- board text added: "REV A"

Commit message: generated gerbers and re-numbered
Parts:
- renumbered L2 to L1, R3 to R1, R4 to R2, U4 to U3
Changed lines of the file:
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@@
 <setting verticaltext="up"/>
 </settings>
-<grid distance="0.5" unitdist="mm" unit="mm" style="lines" multiple="1" display="yes" altdistance="0.635" altunitdist="mm" altunit="mm"/>
+<grid distance="39.3700787" unitdist="mil" unit="mil" style="lines" multiple="1" display="yes" altdistance="0.635" altunitdist="mm" altunit="mm"/>
 <layers>
 <layer number="1" name="Top" color="4" fill="1" visible="yes" active="yes"/>
@@
 <layer number="27" name="tValues" color="7" fill="1" visible="no" active="yes"/>
 <layer number="28" name="bValues" color="7" fill="1" visible="no" active="yes"/>
-<layer number="29" name="tStop" color="7" fill="3" visible="no" active="yes"/>
+<layer number="29" name="tStop" color="7" fill="3" visible="yes" active="yes"/>
 <layer number="30" name="bStop" color="7" fill="6" visible="no" active="yes"/>
 <layer number="31" name="tCream" color="7" fill="4" visible="no" active="yes"/>
@@
 <attribute name="VALUE" x="30.495" y="16.685" size="0.8128" layer="27" ratio="10" rot="R90"/>
 </element>
-<element name="U4" library="Maxim_By_element14_Batch_1" package="SOT95P228X119-3N" value="MAX6326UR29+" x="22.74" y="18.44" smashed="yes">
+<element name="U3" library="Maxim_By_element14_Batch_1" package="SOT95P228X119-3N" value="MAX6326UR29+" x="22.74" y="18.44" smashed="yes">
 <attribute name="PACKAGE" value="SOT-23-3" x="22.74" y="18.44" size="1.778" layer="27" display="off"/>
 <attribute name="OC_NEWARK" value="-" x="22.74" y="18.44" size="1.778" layer="27" display="off"/>
@@
 <attribute name="DIGIKEY" value="CP-002AHPJCT-ND" x="2.31" y="7.82" size="1.778" layer="27" display="off"/>
 </element>
-<element name="L2" library="inductor-tdk" package="VLF302510MT" value="VLF302510MT" x="18.16" y="21.79" smashed="yes" rot="R270">
+<element name="L1" library="inductor-tdk" package="VLF302510MT" value="VLF302510MT" x="18.16" y="21.79" smashed="yes" rot="R270">
 <attribute name="DIGIKEY" value="445-6775-1-ND" x="18.16" y="21.79" size="1.778" layer="27" rot="R270" display="off"/>
 <attribute name="NAME" x="20.311" y="22.941" size="1.016" layer="25" font="vector" ratio="12" rot="R270"/>
 <attribute name="VALUE" x="15.747" y="23.441" size="0.8128" layer="27" ratio="10" rot="R270"/>
 </element>
-<element name="R3" library="Yageo_By_element14_Batch_1" package="RESC1608X60N" value="100K Ohms" x="10.85" y="19.48" smashed="yes" rot="R90">
+<element name="R1" library="Yageo_By_element14_Batch_1" package="RESC1608X60N" value="100K Ohms" x="10.85" y="19.48" smashed="yes" rot="R90">
 <attribute name="OC_NEWARK" value="98K7287" x="10.85" y="19.48" size="1.778" layer="27" rot="R90" display="off"/>
 <attribute name="TOLERANCE" value="±5%" x="10.85" y="19.48" size="1.778" layer="27" rot="R90" display="off"/>
@@
 <attribute name="VALUE" x="14.025" y="16.0256" size="2.0828" layer="27" ratio="10" rot="SR90"/>
 </element>
-<element name="R4" library="Yageo_By_element14_Batch_1" package="RESC1608X60N" value="100K Ohms" x="8.27" y="21.79" smashed="yes" rot="R90">
+<element name="R2" library="Yageo_By_element14_Batch_1" package="RESC1608X60N" value="100K Ohms" x="8.27" y="21.79" smashed="yes" rot="R90">
 <attribute name="OC_NEWARK" value="98K7287" x="8.27" y="21.79" size="1.778" layer="27" rot="R90" display="off"/>
 <attribute name="TOLERANCE" value="±5%" x="8.27" y="21.79" size="1.778" layer="27" rot="R90" display="off"/>
@@
 <contactref element="U2" pad="2"/>
 <contactref element="C1" pad="2"/>
-<contactref element="U4" pad="1"/>
-<contactref element="R4" pad="2"/>
+<contactref element="U3" pad="1"/>
+<contactref element="R2" pad="2"/>
 <contactref element="BATTERY" pad="P4"/>
 <wire x1="21.5716" y1="19.3798" x2="19.9018" y2="17.71" width="0.4064" layer="1"/>
@@
 <signal name="SW1">
 <contactref element="U2" pad="6"/>
-<contactref element="L2" pad="2"/>
+<contactref element="L1" pad="2"/>
 <wire x1="15.2898" y1="20.647" x2="15.5468" y2="20.39" width="0.4064" layer="1"/>
 <wire x1="15.5468" y1="20.39" x2="18.16" y2="20.39" width="0.4064" layer="1"/>
@@
 <signal name="SW2">
 <contactref element="U2" pad="1"/>
-<contactref element="L2" pad="1"/>
+<contactref element="L1" pad="1"/>
 <wire x1="18.16" y1="23.19" x2="17.903" y2="22.933" width="0.4064" layer="1"/>
 <wire x1="17.903" y1="22.933" x2="15.2898" y2="22.933" width="0.4064" layer="1"/>
@@
 <signal name="!SHDN">
 <contactref element="U2" pad="4"/>
-<contactref element="R3" pad="2"/>
+<contactref element="R1" pad="2"/>
 <wire x1="10.85" y1="20.3182" x2="11.1788" y2="20.647" width="0.4064" layer="1"/>
 <wire x1="11.1788" y1="20.647" x2="13.4102" y2="20.647" width="0.4064" layer="1"/>
 </signal>
 <signal name="N$1">
-<contactref element="U4" pad="2"/>
+<contactref element="U3" pad="2"/>
 <contactref element="Q1" pad="1"/>
 <wire x1="21.5716" y1="17.5002" x2="28.2802" y2="17.5002" width="0.4064" layer="1"/>
@@
 <contactref element="J2" pad="VIN0"/>
 <contactref element="D1" pad="P$1"/>
-<contactref element="U4" pad="3"/>
-<contactref element="R4" pad="1"/>
+<contactref element="U3" pad="3"/>
+<contactref element="R2" pad="1"/>
 <wire x1="23.9084" y1="18.44" x2="23.9084" y2="20.9416" width="0.4064" layer="1"/>
 <wire x1="23.9084" y1="20.9416" x2="22.51" y2="22.34" width="0.4064" layer="1"/>
@@
 <contactref element="C1" pad="1"/>
 <contactref element="Q1" pad="2"/>
-<contactref element="R3" pad="1"/>
+<contactref element="R1" pad="1"/>
 <wire x1="28.42" y1="19.54" x2="28.42" y2="23.08" width="0.4064" layer="1"/>
 <wire x1="28.42" y1="23.08" x2="25" y2="26.5" width="0.4064" layer="1"/>

Commit message: started running brad's python scripts
Parts:
- renumbered J2 to J1
Changed lines of the file:
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@@
 <attribute name="VALUE" x="19.2856" y="13.995" size="2.0828" layer="27" ratio="10" rot="SR0"/>
 </element>
-<element name="J2" library="SparkFun-Connectors" package="POWER_JACK_SMD" value="5.5x2.1mm Barrel" x="2.31" y="7.82">
+<element name="J1" library="SparkFun-Connectors" package="POWER_JACK_SMD" value="5.5x2.1mm Barrel" x="2.31" y="7.82">
 <attribute name="SF_ID" value="PRT-12748" x="2.31" y="7.82" size="1.778" layer="27" display="off"/>
 <attribute name="PROD_ID" value="CONN-08106" x="2.31" y="7.82" size="1.778" layer="27" display="off"/>
@@
 <vertex x="9.5" y="27.5"/>
 </polygon>
-<contactref element="J2" pad="GND"/>
-<contactref element="J2" pad="P$4"/>
+<contactref element="J1" pad="GND"/>
+<contactref element="J1" pad="P$4"/>
 <wire x1="2.31" y1="2.12" x2="8.41" y2="2.12" width="0.4064" layer="1"/>
 <wire x1="88.993" y1="6.822" x2="88.808" y2="6.822" width="0.4064" layer="1"/>
@@
 </signal>
 <signal name="N$2">
-<contactref element="J2" pad="VIN0"/>
+<contactref element="J1" pad="VIN0"/>
 <contactref element="D1" pad="P$1"/>
 <contactref element="U3" pad="3"/>
