File: hardware/pcb/eink_schematic.sch (EAGLE design)
At the start: 13 parts, among them J2 5.5x2.1mm Barrel, Q1 FDN340P, U1 NUCLEUM, U2 LTC3531ES6-3PBF, U4 MAX6326UR29+

Commit message: redid battery
Parts:
- added LOGO1: UMICH_SOLID_LARGE, logos:UMICH_SOLID_LARGE
Connections:
- net ENABLE renamed !ENABLE
- net TC_BUSY renamed !TC_BUSY
- removed net N$6: J2.GND, J2.GNDBREAK
- net GND: now also BATTERY.-, J2.GND, J2.GNDBREAK; no longer BATTERY.P4-
- net N$4: now also BATTERY.+; no longer BATTERY.P3+
Changed lines of the file:
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@@
 <attribute name="DIGIKEY" value="36-2462-ND"/>
 </part>
+<part name="LOGO1" library="logos" deviceset="UMICH_SOLID" device="_LARGE"/>
+<part name="GND5" library="umich" deviceset="GND" device=""/>
 </parts>
 <sheets>
@@
 <attribute name="DIGIKEY" x="86.36" y="17.78" size="1.778" layer="96" display="off"/>
 </instance>
+<instance part="LOGO1" gate="G$1" x="45.72" y="35.56"/>
+<instance part="GND5" gate="1" x="33.02" y="93.98"/>
 </instances>
 <busses>
 </busses>
 <nets>
-<net name="TC_BUSY" class="0">
+<net name="!TC_BUSY" class="0">
 <segment>
 <pinref part="U1" gate="G$1" pin="P23"/>
@@
 </segment>
 </net>
-<net name="ENABLE" class="0">
+<net name="!ENABLE" class="0">
 <segment>
 <pinref part="U1" gate="G$1" pin="P24"/>
@@
 </segment>
 <segment>
-<pinref part="BATTERY" gate="KE2462" pin="P4-"/>
+<pinref part="BATTERY" gate="KE2462" pin="-"/>
 <wire x1="111.76" y1="20.32" x2="114.3" y2="20.32" width="0.1524" layer="91"/>
 <wire x1="114.3" y1="20.32" x2="114.3" y2="30.48" width="0.1524" layer="91"/>
@@
 <wire x1="114.3" y1="30.48" x2="119.38" y2="30.48" width="0.1524" layer="91"/>
 <wire x1="119.38" y1="30.48" x2="119.38" y2="25.4" width="0.1524" layer="91"/>
+</segment>
+<segment>
+<pinref part="J2" gate="G$1" pin="GNDBREAK"/>
+<wire x1="38.1" y1="101.6" x2="40.64" y2="101.6" width="0.1524" layer="91"/>
+<wire x1="40.64" y1="101.6" x2="40.64" y2="99.06" width="0.1524" layer="91"/>
+<pinref part="J2" gate="G$1" pin="GND"/>
+<wire x1="40.64" y1="99.06" x2="38.1" y2="99.06" width="0.1524" layer="91"/>
+<wire x1="40.64" y1="99.06" x2="40.64" y2="96.52" width="0.1524" layer="91"/>
+<junction x="40.64" y="99.06"/>
+<pinref part="GND5" gate="1" pin="GND"/>
+<wire x1="40.64" y1="96.52" x2="33.02" y2="96.52" width="0.1524" layer="91"/>
 </segment>
 </net>
@@
 </segment>
 </net>
-<net name="N$6" class="0">
-<segment>
-<pinref part="J2" gate="G$1" pin="GNDBREAK"/>
-<wire x1="38.1" y1="101.6" x2="40.64" y2="101.6" width="0.1524" layer="91"/>
-<wire x1="40.64" y1="101.6" x2="40.64" y2="99.06" width="0.1524" layer="91"/>
-<pinref part="J2" gate="G$1" pin="GND"/>
-<wire x1="40.64" y1="99.06" x2="38.1" y2="99.06" width="0.1524" layer="91"/>
-</segment>
-</net>
 <net name="N$4" class="0">
 <segment>
@@
 <wire x1="86.36" y1="63.5" x2="76.2" y2="63.5" width="0.1524" layer="91"/>
 <wire x1="76.2" y1="63.5" x2="76.2" y2="20.32" width="0.1524" layer="91"/>
-<pinref part="BATTERY" gate="KE2462" pin="P3+"/>
+<pinref part="BATTERY" gate="KE2462" pin="+"/>
 <wire x1="76.2" y1="20.32" x2="81.28" y2="20.32" width="0.1524" layer="91"/>
 </segment>

Commit message: generated gerbers and re-numbered
Parts:
- renumbered L2 to L1, R3 to R1, R4 to R2, U4 to U3
Changed lines of the file:
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@@
 <attribute name="DIGIKEY" value="FDN340PCT-ND"/>
 </part>
-<part name="U4" library="Maxim_By_element14_Batch_1" deviceset="MAX6326UR29+" device="">
+<part name="U3" library="Maxim_By_element14_Batch_1" deviceset="MAX6326UR29+" device="">
 <attribute name="DIGIKEY" value="MAX6326UR29+TCT-ND"/>
 </part>
@@
 </part>
 <part name="GND4" library="umich" deviceset="GND" device=""/>
-<part name="L2" library="inductor-tdk" deviceset="VLF302510MT" device="">
+<part name="L1" library="inductor-tdk" deviceset="VLF302510MT" device="">
 <attribute name="DIGIKEY" value="445-6775-1-ND"/>
 </part>
-<part name="R3" library="Yageo_By_element14_Batch_1" deviceset="RC0603JR-07100KL" device="" value="100K Ohms">
+<part name="R1" library="Yageo_By_element14_Batch_1" deviceset="RC0603JR-07100KL" device="" value="100K Ohms">
 <attribute name="DIGIKEY" value="311-100KGRCT-ND"/>
 </part>
-<part name="R4" library="Yageo_By_element14_Batch_1" deviceset="RC0603JR-07100KL" device="" value="100K Ohms"/>
+<part name="R2" library="Yageo_By_element14_Batch_1" deviceset="RC0603JR-07100KL" device="" value="100K Ohms"/>
 <part name="BATTERY" library="through_hole_battery_pack" deviceset="KEYSTONEELECTRONICS2462" device="">
 <attribute name="DIGIKEY" value="36-2462-ND"/>
@@
 <attribute name="DIGIKEY" x="91.44" y="63.5" size="1.778" layer="96" rot="MR270" display="off"/>
 </instance>
-<instance part="U4" gate="A" x="76.2" y="86.36">
+<instance part="U3" gate="A" x="76.2" y="86.36">
 <attribute name="DIGIKEY" x="76.2" y="86.36" size="1.778" layer="96" display="off"/>
 </instance>
@@
 </instance>
 <instance part="GND4" gate="1" x="50.8" y="68.58"/>
-<instance part="L2" gate="G$1" x="43.18" y="147.32" rot="R90">
+<instance part="L1" gate="G$1" x="43.18" y="147.32" rot="R90">
 <attribute name="DIGIKEY" x="43.18" y="147.32" size="1.778" layer="96" rot="R90" display="off"/>
 </instance>
-<instance part="R3" gate="A" x="55.88" y="152.4" rot="R90">
+<instance part="R1" gate="A" x="55.88" y="152.4" rot="R90">
 <attribute name="DIGIKEY" x="55.88" y="152.4" size="1.778" layer="96" rot="R90" display="off"/>
 </instance>
-<instance part="R4" gate="A" x="43.18" y="81.28" rot="R90"/>
+<instance part="R2" gate="A" x="43.18" y="81.28" rot="R90"/>
 <instance part="BATTERY" gate="KE2462" x="86.36" y="17.78">
 <attribute name="DIGIKEY" x="86.36" y="17.78" size="1.778" layer="96" display="off"/>
@@
 </segment>
 <segment>
-<pinref part="U4" gate="A" pin="GND"/>
+<pinref part="U3" gate="A" pin="GND"/>
 <wire x1="58.42" y1="81.28" x2="50.8" y2="81.28" width="0.1524" layer="91"/>
 <pinref part="GND4" gate="1" pin="GND"/>
 <wire x1="50.8" y1="81.28" x2="50.8" y2="78.74" width="0.1524" layer="91"/>
-<pinref part="R4" gate="A" pin="R2"/>
+<pinref part="R2" gate="A" pin="R2"/>
 <wire x1="50.8" y1="78.74" x2="50.8" y2="71.12" width="0.1524" layer="91"/>
 <wire x1="43.18" y1="81.28" x2="43.18" y2="78.74" width="0.1524" layer="91"/>
@@
 <pinref part="U2" gate="A" pin="SW1"/>
 <wire x1="48.26" y1="147.32" x2="63.5" y2="147.32" width="0.1524" layer="91"/>
-<pinref part="L2" gate="G$1" pin="2"/>
+<pinref part="L1" gate="G$1" pin="2"/>
 <wire x1="43.18" y1="154.94" x2="43.18" y2="152.4" width="0.1524" layer="91"/>
 </segment>
@@
 <pinref part="U2" gate="A" pin="SW2"/>
 <wire x1="48.26" y1="144.78" x2="63.5" y2="144.78" width="0.1524" layer="91"/>
-<pinref part="L2" gate="G$1" pin="1"/>
+<pinref part="L1" gate="G$1" pin="1"/>
 <wire x1="43.18" y1="139.7" x2="43.18" y2="142.24" width="0.1524" layer="91"/>
 </segment>
@@
 <pinref part="U2" gate="A" pin="~SHDN"/>
 <wire x1="63.5" y1="149.86" x2="55.88" y2="149.86" width="0.1524" layer="91"/>
-<pinref part="R3" gate="A" pin="R2"/>
+<pinref part="R1" gate="A" pin="R2"/>
 <wire x1="55.88" y1="152.4" x2="55.88" y2="149.86" width="0.1524" layer="91"/>
 </segment>
@@
 <net name="N$1" class="0">
 <segment>
-<pinref part="U4" gate="A" pin="~RESET"/>
+<pinref part="U3" gate="A" pin="~RESET"/>
 <pinref part="Q1" gate="G$1" pin="G"/>
 <wire x1="93.98" y1="86.36" x2="93.98" y2="68.58" width="0.1524" layer="91"/>
@@
 <pinref part="J2" gate="G$1" pin="PWR"/>
 <pinref part="D1" gate="G$1" pin="1"/>
-<pinref part="U4" gate="A" pin="VCC"/>
+<pinref part="U3" gate="A" pin="VCC"/>
 <wire x1="38.1" y1="104.14" x2="43.18" y2="104.14" width="0.1524" layer="91"/>
 <wire x1="43.18" y1="104.14" x2="53.34" y2="104.14" width="0.1524" layer="91"/>
@@
 <wire x1="53.34" y1="86.36" x2="53.34" y2="104.14" width="0.1524" layer="91"/>
 <junction x="53.34" y="104.14"/>
-<pinref part="R4" gate="A" pin="R1"/>
+<pinref part="R2" gate="A" pin="R1"/>
 <wire x1="43.18" y1="93.98" x2="43.18" y2="104.14" width="0.1524" layer="91"/>
 <junction x="43.18" y="104.14"/>
@@
 <wire x1="101.6" y1="63.5" x2="101.6" y2="86.36" width="0.1524" layer="91"/>
 <junction x="101.6" y="86.36"/>
-<pinref part="R3" gate="A" pin="R1"/>
+<pinref part="R1" gate="A" pin="R1"/>
 <wire x1="55.88" y1="165.1" x2="55.88" y2="167.64" width="0.1524" layer="91"/>
 <junction x="55.88" y="167.64"/>

Commit message: started running brad's python scripts
Parts:
- renumbered J2 to J1
Changed lines of the file:
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@@
 <attribute name="DIGIKEY" value="MAX6326UR29+TCT-ND"/>
 </part>
-<part name="J2" library="SparkFun-Connectors" deviceset="POWER_JACK" device="SMD" value="5.5x2.1mm Barrel">
+<part name="J1" library="SparkFun-Connectors" deviceset="POWER_JACK" device="SMD" value="5.5x2.1mm Barrel">
 <attribute name="DIGIKEY" value="CP-002AHPJCT-ND"/>
 </part>
@@
 <attribute name="DIGIKEY" x="76.2" y="86.36" size="1.778" layer="96" display="off"/>
 </instance>
-<instance part="J2" gate="G$1" x="35.56" y="96.52">
+<instance part="J1" gate="G$1" x="35.56" y="96.52">
 <attribute name="DIGIKEY" x="35.56" y="96.52" size="1.778" layer="96" display="off"/>
 </instance>
@@
 </segment>
 <segment>
-<pinref part="J2" gate="G$1" pin="GNDBREAK"/>
+<pinref part="J1" gate="G$1" pin="GNDBREAK"/>
 <wire x1="38.1" y1="101.6" x2="40.64" y2="101.6" width="0.1524" layer="91"/>
 <wire x1="40.64" y1="101.6" x2="40.64" y2="99.06" width="0.1524" layer="91"/>
-<pinref part="J2" gate="G$1" pin="GND"/>
+<pinref part="J1" gate="G$1" pin="GND"/>
 <wire x1="40.64" y1="99.06" x2="38.1" y2="99.06" width="0.1524" layer="91"/>
 <wire x1="40.64" y1="99.06" x2="40.64" y2="96.52" width="0.1524" layer="91"/>
@@
 <net name="N$2" class="0">
 <segment>
-<pinref part="J2" gate="G$1" pin="PWR"/>
+<pinref part="J1" gate="G$1" pin="PWR"/>
 <pinref part="D1" gate="G$1" pin="1"/>
 <pinref part="U3" gate="A" pin="VCC"/>
